File: hw/M484/vsf_m484.kicad_pcb (KiCad board)
At the start: 4 copper layers, 34.9 x 30.5 mm, 82 parts, among them J1 Conn_02x10_Odd_Even, J2 USB_B_Micro, J3 USB_A, J4 USB_B_Micro, J5 Conn_01x05, J6 Conn_02x05_Odd_Even, SW0 SW_DIP_x01, U0 M4842U_64, U1 AP1117-33, U2 GD25Q_8P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

Commit message: update to the latest dev repo
Parts:
- removed F0: Fuse, Fuse:Fuse_0805_2012Metric
- J1: footprint SimonQian:PinSocket_2x10_P2.54mm_Horizontal_2Layer -> SimonQian:PinSocket_2x10_P2.54mm_Horizontal_2Layer_NoSilks
Connections:
- J3 pad 1: Net-(F0-Pad2) -> /USBD_VBUS
Routing:
- net Net-(F0-Pad2): track 3.45 -> 0.00 mm
- net /USBD_VBUS: track 57.6 -> 58.7 mm
Other:
- board text added: "3.3V"
- board text added: "5V"
- board text added: "PB0"
- board text added: "PB1"
- board text added: "PB10"
- board text added: "PB11"
- board text added: "PB12"
- board text added: "PB13"
- board text added: "PB14"
- board text added: "PB15"
- board text added: "PB2"
- board text added: "PB3"
- board text added: "PB4"
- board text added: "PB5"
- board text added: "PB6"
- board text added: "PB7"
- board text added: "PB8"
- board text added: "PB9"
