File: hardware/AIC8800/vsf_aic8800.kicad_pcb (KiCad board)
At the start: 2 copper layers, 27.9 x 50.8 mm, 33 parts, among them J0 USB_C_Receptacle_USB2.0, J1 Conn_01x20, J2 Conn_01x20, J3 Conn_02x05_Counter_Clockwise, Q0 AO3401, Q1 AO3402, SW0 SW_Push, SW1 SW_Push, U0 Module_AIC8800M

Commit message: [hardware/aic8800] add board/data silks
Other:
- board text added: "22.0328"
- board text added: "VSF_AIC8800M"
