File: hardware/AIC8800/uikit/uikit.kicad_sch (KiCad schematic)
At the start: 26 parts, among them J0 Micro_SD_Card, J1 Conn_01x20, J1 PJ-393-USA, J2 Conn_01x20, J3 Conn_01x10, J4 Conn_01x06, U0 AIC1000A

Commit message: [hardware/AIC8800/uikit] update
Connections:
- net LCD_RS is gone; now on net A4: J3.10 (Pin_10)

Commit message: [hardware/AIC8800/uikit] update
Connections:
- net B3 is gone; now on net AU_SLEEP: J1.9 (Pin_9)
- net B5 is gone; now on net AU_PWR: J1.17 (Pin_17)
- net CTP_INT is gone; now on net B2: J4.3 (Pin_3), R1.2
- net CTP_RST is gone; now on net B1: J4.2 (Pin_2), R0.2
- net I2C_SCL is gone; now on net A6: J4.5 (Pin_5), R3.2, U0.12 (P_SCL)
- net I2C_SDA is gone; now on net A7: J4.4 (Pin_4), R2.2, U0.11 (P_SDA)
- net JACK_DET is gone; now on net B4: R9.2
- net LCD_RST is gone; now on net B0: J3.6 (Pin_6)
- net A1: now also U0.10 (S_BCK); no longer J3.5 (Pin_5)
- net A7: no longer U0.10 (S_BCK)
- net B13: now also J3.5 (Pin_5)
Changed lines of the file:
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@@
+    (effects (font (size 1.27 1.27)) (justify left bottom))
+  )
+  (label "B13" (at 31.75 86.995 0)
     (effects (font (size 1.27 1.27)) (justify left bottom))
   )
@@
     (effects (font (size 1.27 1.27)) (justify right bottom))
   )
+  (label "B1" (at 31.75 94.615 0)
+    (effects (font (size 1.27 1.27)) (justify left bottom))
+  )
+  (label "B5" (at 31.75 137.795 0)
+    (effects (font (size 1.27 1.27)) (justify left bottom))
+  )
   (label "CTP_RST" (at 100.965 29.21 180)
     (effects (font (size 1.27 1.27)) (justify right bottom))
@@
     (effects (font (size 1.27 1.27)) (justify right bottom))
   )
+  (label "B2" (at 31.75 97.155 0)
+    (effects (font (size 1.27 1.27)) (justify left bottom))
+  )
   (label "USB_DM" (at 31.75 29.21 0)
     (effects (font (size 1.27 1.27)) (justify left bottom))
@@
     (effects (font (size 1.27 1.27)) (justify right bottom))
   )
-  (label "A1" (at 31.75 86.995 0)
+  (label "A1" (at 31.75 120.015 0)
     (effects (font (size 1.27 1.27)) (justify left bottom))
   )
@@
     (effects (font (size 1.27 1.27)) (justify left bottom))
   )
-  (label "A7" (at 31.75 120.015 0)
-    (effects (font (size 1.27 1.27)) (justify left bottom))
-  )
   (label "TF_CMD" (at 127 36.83 180)
     (effects (font (size 1.27 1.27)) (justify right bottom))
@@
     (effects (font (size 1.27 1.27)) (justify left bottom))
   )
+  (label "A7" (at 31.75 99.695 0)
+    (effects (font (size 1.27 1.27)) (justify left bottom))
+  )
   (label "I2C_SDA" (at 100.965 34.29 180)
     (effects (font (size 1.27 1.27)) (justify right bottom))
@@
     (effects (font (size 1.27 1.27)) (justify right bottom))
   )
+  (label "B3" (at 31.75 132.715 0)
+    (effects (font (size 1.27 1.27)) (justify left bottom))
+  )
   (label "VCC" (at 125.095 81.28 0)
     (effects (font (size 1.27 1.27)) (justify left bottom))
@@
     (effects (font (size 1.27 1.27)) (justify right bottom))
   )
+  (label "B0" (at 31.75 92.075 0)
+    (effects (font (size 1.27 1.27)) (justify left bottom))
+  )
   (label "HP_R+" (at 139.7 129.54 180)
     (effects (font (size 1.27 1.27)) (justify right bottom))
@@
     (effects (font (size 1.27 1.27)) (justify right bottom))
   )
+  (label "A6" (at 31.75 102.235 0)
+    (effects (font (size 1.27 1.27)) (justify left bottom))
+  )
   (label "I2S_BCK" (at 92.075 106.68 270)
     (effects (font (size 1.27 1.27)) (justify right bottom))
@@
     (effects (font (size 1.27 1.27)) (justify right bottom))
   )
+  (label "B4" (at 31.75 135.255 0)
+    (effects (font (size 1.27 1.27)) (justify left bottom))
+  )
   (label "B6" (at 31.75 69.85 0)

Commit message: [hardware/AIC8800/uikit] ad CH340N
Parts:
- added C8: 0.1uF, symbol Device:C
- added D0: LESD5Z5.0CT1G, Diode_SMD:D_SOD-523, symbol Device:D_TVS
- added J6: USB_C_Receptacle_USB2.0, simonqian:USB_C_Receptacle_Palconn_UTC16-G_DOWN1.6, symbol Connector:USB_C_Receptacle_USB2.0
- added R10, R11: 5.1K, Resistor_SMD:R_0402_1005Metric, symbol Device:R
- added R12: 0, Resistor_SMD:R_0402_1005Metric, symbol Device:R
- added R8, R9: 22, Resistor_SMD:R_0402_1005Metric, symbol Device:R
- added U1: CH340N, symbol VSF:CH340N
- renumbered J1 to J5
Connections:
- net B6: now also U1.6 (TXD)
- net B7: now also U1.7 (RXD)
- net GND: now also C8.2, D0.2 (A2), J6.A1 (GND), J6.A12 (GND), J6.A8 (SBU1), J6.B1 (GND), J6.B12 (GND), J6.B8 (SBU2), R10.1, R11.1, R12.1, U1.3 (GND)
- net USB_5V: now also D0.1 (A1), J6.A4 (VBUS), J6.A9 (VBUS), J6.B4 (VBUS), J6.B9 (VBUS)
- net V33: now also C8.1, U1.5 (VCC), U1.8 (V3)
- new net: R8.1, U1.1 (UD+)
- new net: R9.1, U1.2 (UD-)
- new net: J6.A7 (D-), J6.B7 (D-), R8.2
- new net: J6.A5 (CC1), R10.2
- new net: J6.B5 (CC2), R11.2
- new net: J6.S1 (SHIELD), R12.2
- new net: J6.A6 (D+), J6.B6 (D+), R9.2
Other:
- moved on the sheet: C6, C7, C8, J0, J4, J5, R0, R1, R2, R3, R8, R9

Commit message: [hardware/AIC8800/uikit] update
Parts:
- added R13: NC, symbol Device:R
Connections:
- net BL_K is gone; now on net GND: J3.8 (Pin_8)
- net BL_A: now also R13.1
- net V33: now also R13.2
Other:
- moved on the sheet: J3, J4, R0, R1, R2, R3

Commit message: [hardware/AIC8800/uikit] update
Parts:
- added R14: 10K, symbol Device:R
- R2, R3: value 10K -> 4.7K
Connections:
- net A6: no longer U0.12 (P_SCL)
- net A7: no longer U0.11 (P_SDA)
- net GND: now also J3.5 (Pin_5)
- net V33: now also R14.2
- net B0 renamed AU_SCL
- net AU_SCL: now also U0.12 (P_SCL); no longer J3.6 (Pin_6)
- net B13 renamed AU_SDA
- net AU_SDA: now also U0.11 (P_SDA); no longer J3.5 (Pin_5)
- new net LCD_RST: J3.6 (Pin_6), R14.1
Other:
- moved on the sheet: J3, R13

Commit message: [hardware/AIC8800/uikit] update
Parts:
- removed R14: 10K, symbol Device:R
Connections:
- net LCD_RST is gone; now on net B1: J3.6 (Pin_6)
Changed lines of the file:
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@@
-    (stroke (width 0) (type default) (color 0 0 0 0))
-  )
-  (wire (pts (xy 61.595 39.37) (xy 68.58 39.37))
     (stroke (width 0) (type default) (color 0 0 0 0))
   )
@@
     (effects (font (size 1.27 1.27)) (justify right bottom))
   )
-  (label "V33" (at 61.595 39.37 0)
-    (effects (font (size 1.27 1.27)) (justify left bottom))
-  )
   (label "TF_CMD" (at 48.26 109.855 180)
     (effects (font (size 1.27 1.27)) (justify right bottom))
@@
   )
   (label "A6" (at 31.75 102.235 0)
+    (effects (font (size 1.27 1.27)) (justify left bottom))
+  )
+  (label "B1" (at 31.75 92.075 0)
     (effects (font (size 1.27 1.27)) (justify left bottom))
   )
@@
     )
     (property "Datasheet" "~" (id 3) (at 157.48 79.375 0)
-      (effects (font (size 1.27 1.27)) hide)
-    )
-    (pin "1")
-    (pin "2")
-  )
-  (symbol (lib_id "Device:R") (at 72.39 39.37 270) (unit 1)
-    (in_bom yes) (on_board yes)
-    (property "Reference" "R14" (id 0) (at 66.04 38.1 90)
-      (effects (font (size 1.27 1.27)) (justify left))
-    )
-    (property "Value" "10K" (id 1) (at 70.485 39.37 90)
-      (effects (font (size 1.27 1.27)) (justify left))
-    )
-    (property "Footprint" "" (id 2) (at 72.39 37.592 90)
-      (effects (font (size 1.27 1.27)) hide)
-    )
-    (property "Datasheet" "~" (id 3) (at 72.39 39.37 0)
       (effects (font (size 1.27 1.27)) hide)
     )
@@
   (symbol (lib_id "Device:R") (at 72.39 41.91 270) (unit 1)
     (in_bom yes) (on_board yes)
-    (property "Reference" "R13" (id 0) (at 66.04 43.18 90)
+    (property "Reference" "R13" (id 0) (at 70.485 39.37 90)
       (effects (font (size 1.27 1.27)) (justify left))
     )
@@
       (reference "R13") (unit 1) (value "NC") (footprint "")
     )
-    (path "/4e28c148-3338-4282-a698-8659286d610b"
-      (reference "R14") (unit 1) (value "10K") (footprint "")
-    )
     (path "/ab0bba3b-9902-471a-8615-9dfda2c848da"

Commit message: [hardware/AIC8800/uikit] prepare pcb
Parts:
- removed J5: PJ-393-USA, symbol VSF:PJ-393-USA
- added J7: PJ-393-USA, VSF:PJ-393, symbol VSF:PJ-393-USA
- C1: footprint (none) -> Capacitor_SMD:C_0402_1005Metric
- C10, C7: renamed from C8; footprint (none) -> Capacitor_SMD:C_0402_1005Metric
- C2: renamed from C0; footprint (none) -> Capacitor_SMD:C_0402_1005Metric
- C3: renamed from C2; footprint (none) -> Capacitor_SMD:C_0402_1005Metric
- C4: renamed from C3; footprint (none) -> Capacitor_SMD:C_0402_1005Metric
- C5: renamed from C4; footprint (none) -> Capacitor_SMD:C_0402_1005Metric
- C6: renamed from C5; footprint (none) -> Capacitor_SMD:C_0402_1005Metric
- C8: renamed from C7; footprint (none) -> Capacitor_SMD:C_0402_1005Metric
- C9: renamed from C6; footprint (none) -> Capacitor_SMD:C_0402_1005Metric
- J3: footprint (none) -> Connector_FFC-FPC:Hirose_FH12-10S-0.5SH_1x10-1MP_P0.50mm_Horizontal
- J4: footprint (none) -> Connector_FFC-FPC:Hirose_FH12-6S-0.5SH_1x06-1MP_P0.50mm_Horizontal
- J5: renamed from J6; footprint simonqian:USB_C_Receptacle_Palconn_UTC16-G_DOWN1.6 -> VSF:USB_C_Receptacle_Palconn_UTC16-G_DOWN1.6
- J6: renamed from J0; footprint (none) -> Connector_Card:microSD_HC_Wuerth_693072010801
- R1: renamed from R13; footprint (none) -> Resistor_SMD:R_1206_3216Metric
- R10: renamed from R4; footprint (none) -> Resistor_SMD:R_0402_1005Metric
- R15: renamed from R8; footprint (none) -> Resistor_SMD:R_0402_1005Metric
- R16: renamed from R9; footprint (none) -> Resistor_SMD:R_0402_1005Metric
- R2: renamed from R3; footprint (none) -> Resistor_SMD:R_0402_1005Metric
- R3: renamed from R2; footprint (none) -> Resistor_SMD:R_0402_1005Metric
- R4: renamed from R1; footprint (none) -> Resistor_SMD:R_0402_1005Metric
- R5: renamed from R0; footprint (none) -> Resistor_SMD:R_0402_1005Metric
- R7: footprint (none) -> Resistor_SMD:R_0402_1005Metric
- R8: renamed from R6; footprint (none) -> Resistor_SMD:R_0402_1005Metric
- R9: renamed from R5; footprint (none) -> Resistor_SMD:R_0402_1005Metric
- U1: renamed from U0; footprint (none) -> Package_DFN_QFN:QFN-24-1EP_3x4mm_P0.4mm_EP1.65x2.65mm
- U2: renamed from U1; footprint (none) -> Package_SO:SOP-8_3.9x4.9mm_P1.27mm
- renumbered D0 to D1, R10 to R11, R11 to R12, R8 to R13, R9 to R14, R12 to R6
Connections:
- net GND: now also J7.7
- net at C9.2: now also J7.2, J7.5
- net at C7.2, R15.1: now also J7.1, J7.8
- net at C8.2: now also J7.3, J7.6
- net at R16.1: now also J7.4

Commit message: [hardware/AIC8800/uikit] add PCB
Connections:
- net GND: now also C4.1, C5.1
Changed lines of the file:
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@@
   (junction (at 161.29 66.675) (diameter 0) (color 0 0 0 0)
   )
+  (junction (at 89.535 123.825) (diameter 0) (color 0 0 0 0)
+  )
   (junction (at 163.83 84.455) (diameter 0) (color 0 0 0 0)
   )
@@
   )
   (wire (pts (xy 145.415 111.76) (xy 149.225 111.76))
+    (stroke (width 0) (type default) (color 0 0 0 0))
+  )
+  (wire (pts (xy 84.455 123.825) (xy 89.535 123.825))
     (stroke (width 0) (type default) (color 0 0 0 0))
   )
@@
   (symbol (lib_id "Device:C") (at 89.535 120.015 180) (unit 1)
     (in_bom yes) (on_board yes)
-    (property "Reference" "C5" (id 0) (at 88.265 123.19 90))
+    (property "Reference" "C5" (id 0) (at 90.805 123.19 90))
     (property "Value" "0.1uF" (id 1) (at 92.71 120.015 90))
     (property "Footprint" "Capacitor_SMD:C_0402_1005Metric" (id 2) (at 88.5698 116.205 0)
@@
     (pin "1")
     (pin "2")
+  )
+  (symbol (lib_id "power:GND") (at 89.535 123.825 0) (unit 1)
+    (in_bom yes) (on_board yes)
+    (property "Reference" "#PWR?" (id 0) (at 89.535 130.175 0)
+      (effects (font (size 1.27 1.27)) hide)
+    )
+    (property "Value" "GND" (id 1) (at 89.662 128.2192 0))
+    (property "Footprint" "" (id 2) (at 89.535 123.825 0)
+      (effects (font (size 1.27 1.27)) hide)
+    )
+    (property "Datasheet" "" (id 3) (at 89.535 123.825 0)
+      (effects (font (size 1.27 1.27)) hide)
+    )
+    (pin "1")
   )
   (symbol (lib_id "Device:R") (at 103.505 32.385 0) (unit 1)
@@
       (reference "#PWR012") (unit 1) (value "GND") (footprint "")
     )
+    (path "/9dd17a99-13f8-4622-803f-81aed440e841"
+      (reference "#PWR?") (unit 1) (value "GND") (footprint "")
+    )
     (path "/faf7f873-d004-44e5-b2bd-9d7562f28cb5"
